Commit message: fix: URDF mesh 引用改为相对路径 ../meshes/，pybullet 跨版本可解析（不改生成脚本）

File: AnyDexGrasp/generate_mesh_and_pointcloud/inspire_urdf/urdf-five3/robots/urdf-five3.urdf (robot description, URDF)
Before this commit: robot urdf-five3, 13 links, 12 joints
Links:
- link Link1: geometry collision mesh filename=../meshes/Link1.STL; visual mesh filename=../meshes/Link1.STL
- link Link11: geometry collision mesh filename=../meshes/Link11.STL; visual mesh filename=../meshes/Link11.STL
- link Link111: geometry collision mesh filename=../meshes/Link111.STL; visual mesh filename=../meshes/Link111.STL
- link Link2: geometry collision mesh filename=../meshes/Link2.STL; visual mesh filename=../meshes/Link2.STL
- link Link22: geometry collision mesh filename=../meshes/Link22.STL; visual mesh filename=../meshes/Link22.STL
- link Link3: geometry collision mesh filename=../meshes/Link3.STL; visual mesh filename=../meshes/Link3.STL
- link Link33: geometry collision mesh filename=../meshes/Link33.STL; visual mesh filename=../meshes/Link33.STL
- link Link4: geometry collision mesh filename=../meshes/Link4.STL; visual mesh filename=../meshes/Link4.STL
- link Link44: geometry collision mesh filename=../meshes/Link44.STL; visual mesh filename=../meshes/Link44.STL
- link Link5: geometry collision mesh filename=../meshes/Link5.STL; visual mesh filename=../meshes/Link5.STL
- link Link51: geometry collision mesh filename=../meshes/Link51.STL; visual mesh filename=../meshes/Link51.STL
- link Link52: geometry collision mesh filename=../meshes/Link52.STL; visual mesh filename=../meshes/Link52.STL
- link Link53: geometry collision mesh filename=../meshes/Link53.STL; visual mesh filename=../meshes/Link53.STL

Commit message: fix: 提交 URDF 链接视觉 mesh(urdf-five3/meshes/*.STL,10M)；收窄 .gitignore 只忽略生成产物。这是目标机 loadURDF 失败的真正根因（STL 缺失），URDF 还原为原版 package://

File: AnyDexGrasp/generate_mesh_and_pointcloud/inspire_urdf/urdf-five3/robots/urdf-five3.urdf (robot description, URDF)
Before this commit: robot urdf-five3, 13 links, 12 joints
Links:
- link Link1: geometry collision mesh filename=package://urdf-five3/meshes/Link1.STL; visual mesh filename=package://urdf-five3/meshes/Link1.STL
- link Link11: geometry collision mesh filename=package://urdf-five3/meshes/Link11.STL; visual mesh filename=package://urdf-five3/meshes/Link11.STL
- link Link111: geometry collision mesh filename=package://urdf-five3/meshes/Link111.STL; visual mesh filename=package://urdf-five3/meshes/Link111.STL
- link Link2: geometry collision mesh filename=package://urdf-five3/meshes/Link2.STL; visual mesh filename=package://urdf-five3/meshes/Link2.STL
- link Link22: geometry collision mesh filename=package://urdf-five3/meshes/Link22.STL; visual mesh filename=package://urdf-five3/meshes/Link22.STL
- link Link3: geometry collision mesh filename=package://urdf-five3/meshes/Link3.STL; visual mesh filename=package://urdf-five3/meshes/Link3.STL
- link Link33: geometry collision mesh filename=package://urdf-five3/meshes/Link33.STL; visual mesh filename=package://urdf-five3/meshes/Link33.STL
- link Link4: geometry collision mesh filename=package://urdf-five3/meshes/Link4.STL; visual mesh filename=package://urdf-five3/meshes/Link4.STL
- link Link44: geometry collision mesh filename=package://urdf-five3/meshes/Link44.STL; visual mesh filename=package://urdf-five3/meshes/Link44.STL
- link Link5: geometry collision mesh filename=package://urdf-five3/meshes/Link5.STL; visual mesh filename=package://urdf-five3/meshes/Link5.STL
- link Link51: geometry collision mesh filename=package://urdf-five3/meshes/Link51.STL; visual mesh filename=package://urdf-five3/meshes/Link51.STL
- link Link52: geometry collision mesh filename=package://urdf-five3/meshes/Link52.STL; visual mesh filename=package://urdf-five3/meshes/Link52.STL
- link Link53: geometry collision mesh filename=package://urdf-five3/meshes/Link53.STL; visual mesh filename=package://urdf-five3/meshes/Link53.STL
